File: eagle/odessa_rev_A.brd (EAGLE design)
At the start: 72 x 42 mm, 30 parts, among them IC1 PIC18F2580, IC3 SN65HVD232, IC4 LM2575S, J2 A00-108-220-450, Q1 10 MHz

Commit message: Fixed bug in control byte write routine
Parts:
- C14: value 1 uF -> 10 uF
Changed lines of the file:
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@@
 <attribute name="VALUE" x="48.91" y="20.07" size="1.27" layer="27" rot="R270"/>
 </element>
-<element name="C14" library="rcl" package="C0805" value="1 uF" x="55.91" y="30.62" smashed="yes" rot="R180">
+<element name="C14" library="rcl" package="C0805" value="10 uF" x="55.91" y="30.62" smashed="yes" rot="R180">
 <attribute name="NAME" x="59.08" y="33.13" size="1.27" layer="25" font="fixed" rot="R180"/>
 </element>
