File: eagle/odessa_rev_A.sch (EAGLE design)
At the start: 30 parts, among them IC1 PIC18F2580, IC3 SN65HVD232, IC4 LM2575S, J2 A00-108-220-450, Q1 10 MHz

Commit message: Fixed bug in control byte write routine
Parts:
- C14: value 1 uF -> 10 uF
Changed lines of the file:
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@@
 <part name="LED2" library="led" deviceset="LED" device="CHIP-LED0805" value="Red LED"/>
 <part name="P+9" library="SUPPLY1" deviceset="VCC" device=""/>
-<part name="C14" library="rcl" deviceset="C-EU" device="C0805" value="1 uF"/>
+<part name="C14" library="rcl" deviceset="C-EU" device="C0805" value="10 uF"/>
 <part name="GND32" library="SUPPLY1" deviceset="GND" device=""/>
 <part name="R17" library="rcl" deviceset="R-EU_" device="R0805" value="120"/>
@@
 <instance part="C14" gate="G$1" x="10.16" y="193.04" smashed="yes" rot="R180">
 <attribute name="NAME" x="8.636" y="192.659" size="1.778" layer="95" rot="R180"/>
-<attribute name="VALUE" x="18.796" y="195.199" size="1.778" layer="96" rot="R180"/>
+<attribute name="VALUE" x="18.796" y="195.199" size="1.778" layer="91" rot="R180"/>
 </instance>
 <instance part="GND32" gate="1" x="10.16" y="182.88"/>
